File: Dice.kicad_sch (KiCad schematic)
At the start: 24 parts, among them Q1 NPN, SW1 SW_Push, U1 LM555xM, U2 4017, U3 74LS32

Commit message: Test
Parts:
- added R12: 300, Package_DIP:DIP-8_W7.62mm, symbol Device:R_US
- R10, R4, R5, R6, R7, R8, R9: value 300 ohm -> 300
- R11: value 100K -> 2K
Connections:
- net +5V: now also R12.2; no longer Q1.1 (C), R10.1, R5.1
- net at R9.1, U3.11: now also R5.1; no longer R4.1
- net at R8.1, U2.1 (Q5), U3.13: now also R6.2; no longer R6.1
- net at D3.2 (A): now also R6.1; no longer R6.2
- new net: Q1.1 (C), R10.1, R12.1, R4.1
Other:
- note added: "LED 1"
- note added: "LED 2 Y 7"
- note added: "LED 3 Y 6"
- note added: "LED 4 y 5"
- moved on the sheet: C1, D1, D2, D3, D4, D5, D6, D7, Q1, R1, R10, R11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

Commit message: Test
Parts:
- added BT1: Battery_Cell, symbol Device:Battery_Cell
- added SW2: SW_DPST_x2, symbol Switch:SW_DPST_x2
- R6, R8: value 300 -> 1k
Connections:
- net GND: now also BT1.2 (-)
- net +5V renamed +3V
- net +3V: now also SW2.2 (B)
- new net: BT1.1 (+), SW2.1 (A)
Other:
- moved on the sheet: D3, D5, D6, D7, R5, R6, R8, R9, U3C, U3D

Commit message: FOOTPRINT ASSIGNED
Parts:
- BT1: footprint (none) -> Battery:BatteryHolder_Keystone_1060_1x2032
- C1: footprint Package_SO:SOIC-8_3.9x4.9mm_P1.27mm -> Capacitor_THT:C_Disc_D5.0mm_W2.5mm_P2.50mm
- D1, D2, D3, D4, D5, D6, D7: footprint (none) -> LED_THT:LED_D5.0mm
- Q1: footprint Package_DIP:DIP-6_W7.62mm -> Package_TO_SOT_THT:TO-92_Inline
- R1, R2, R3: footprint (none) -> Resistor_THT:R_Axial_DIN0204_L3.6mm_D1.6mm_P5.08mm_Horizontal
- R10, R11, R12, R4, R5, R6, R7, R8, R9: footprint Package_DIP:DIP-8_W7.62mm -> Resistor_THT:R_Axial_DIN0204_L3.6mm_D1.6mm_P5.08mm_Horizontal
- SW1: footprint Package_SON:WSON-8-1EP_6x5mm_P1.27mm_EP3.4x4mm -> Button_Switch_THT:SW_PUSH-12mm_Wuerth-430476085716
- SW2: footprint (none) -> Button_Switch_THT:SW_DIP_SPSTx01_Slide_9.78x4.72mm_W7.62mm_P2.54mm
- U1: footprint Package_SO:SOIC-8_3.9x4.9mm_P1.27mm -> Package_DIP:DIP-8_W7.62mm
- U2: footprint Package_TO_SOT_SMD:SOT-363_SC-70-6 -> Package_DIP:DIP-16_W7.62mm
- U3: footprint Package_SO:SSOP-24_5.3x8.2mm_P0.65mm -> Package_DIP:DIP-14_W7.62mm
Changed lines of the file:
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@@
 			)
 		)
-		(property "Footprint" "Package_DIP:DIP-8_W7.62mm"
+		(property "Footprint" "Resistor_THT:R_Axial_DIN0204_L3.6mm_D1.6mm_P5.08mm_Horizontal"
 			(at 204.216 105.664 90)
 			(hide yes)
@@
 			)
 		)
-		(property "Footprint" ""
+		(property "Footprint" "Battery:BatteryHolder_Keystone_1060_1x2032"
 			(at 19.05 23.876 90)
 			(hide yes)
@@
 			)
 		)
-		(property "Footprint" "Package_SO:SSOP-24_5.3x8.2mm_P0.65mm"
+		(property "Footprint" "Package_DIP:DIP-14_W7.62mm"
 			(at 43.18 63.5 0)
 			(hide yes)
@@
 			)
 		)
-		(property "Footprint" ""
+		(property "Footprint" "Button_Switch_THT:SW_DIP_SPSTx01_Slide_9.78x4.72mm_W7.62mm_P2.54mm"
 			(at 35.56 20.32 0)
 			(hide yes)
@@
 			)
 		)
-		(property "Footprint" ""
+		(property "Footprint" "Resistor_THT:R_Axial_DIN0204_L3.6mm_D1.6mm_P5.08mm_Horizontal"
 			(at 143.256 39.624 90)
 			(hide yes)
@@
 			)
 		)
-		(property "Footprint" "Package_DIP:DIP-8_W7.62mm"
+		(property "Footprint" "Resistor_THT:R_Axial_DIN0204_L3.6mm_D1.6mm_P5.08mm_Horizontal"
 			(at 186.436 54.864 90)
 			(hide yes)
@@
 			)
 		)
-		(property "Footprint" "Package_DIP:DIP-8_W7.62mm"
+		(property "Footprint" "Resistor_THT:R_Axial_DIN0204_L3.6mm_D1.6mm_P5.08mm_Horizontal"
 			(at 187.706 137.414 90)
 			(hide yes)
@@
 			)
 		)
-		(property "Footprint" "Package_DIP:DIP-8_W7.62mm"
+		(property "Footprint" "Resistor_THT:R_Axial_DIN0204_L3.6mm_D1.6mm_P5.08mm_Horizontal"
 			(at 143.764 139.446 90)
 			(hide yes)
@@
 			)
 		)
-		(property "Footprint" "Package_DIP:DIP-8_W7.62mm"
+		(property "Footprint" "Resistor_THT:R_Axial_DIN0204_L3.6mm_D1.6mm_P5.08mm_Horizontal"
 			(at 166.624 42.164 90)
 			(hide yes)
@@
 			)
 		)
-		(property "Footprint" "Package_DIP:DIP-6_W7.62mm"
+		(property "Footprint" "Package_TO_SOT_THT:TO-92_Inline"
 			(at 170.18 111.76 0)
 			(hide yes)
@@
 			)
 		)
-		(property "Footprint" "Package_SO:SOIC-8_3.9x4.9mm_P1.27mm"
+		(property "Footprint" "Package_DIP:DIP-8_W7.62mm"
 			(at 49.53 43.18 0)
 			(hide yes)
@@
 			)
 		)
-		(property "Footprint" "Package_DIP:DIP-8_W7.62mm"
+		(property "Footprint" "Resistor_THT:R_Axial_DIN0204_L3.6mm_D1.6mm_P5.08mm_Horizontal"
 			(at 174.244 41.656 90)
 			(hide yes)
@@
 			)
 		)
-		(property "Footprint" "Package_DIP:DIP-8_W7.62mm"
+		(property "Footprint" "Resistor_THT:R_Axial_DIN0204_L3.6mm_D1.6mm_P5.08mm_Horizontal"
 			(at 153.924 139.954 90)
 			(hide yes)
@@
 			)
 		)
-		(property "Footprint" ""
+		(property "Footprint" "LED_THT:LED_D5.0mm"
 			(at 199.39 144.78 0)
 			(hide yes)
@@
 			)
 		)
-		(property "Footprint" "Package_DIP:DIP-8_W7.62mm"
+		(property "Footprint" "Resistor_THT:R_Axial_DIN0204_L3.6mm_D1.6mm_P5.08mm_Horizontal"
 			(at 200.406 137.414 90)
 			(hide yes)
@@
 			)
 		)
-		(property "Footprint" ""
+		(property "Footprint" "LED_THT:LED_D5.0mm"
 			(at 144.78 147.32 0)
 			(hide yes)
@@
 			)
 		)
-		(property "Footprint" "Package_SO:SSOP-24_5.3x8.2mm_P0.65mm"
+		(property "Footprint" "Package_DIP:DIP-14_W7.62mm"
 			(at 175.26 116.84 0)
 			(hide yes)
@@
 			)
 		)
-		(property "Footprint" ""
+		(property "Footprint" "LED_THT:LED_D5.0mm"
 			(at 186.69 144.78 0)
 			(hide yes)
@@
 			)
 		)
-		(property "Footprint" "Package_SON:WSON-8-1EP_6x5mm_P1.27mm_EP3.4x4mm"
+		(property "Footprint" "Button_Switch_THT:SW_PUSH-12mm_Wuerth-430476085716"
 			(at 31.75 46.99 0)
 			(hide yes)
@@
 			)
 		)
-		(property "Footprint" "Package_SO:SSOP-24_5.3x8.2mm_P0.65mm"
+		(property "Footprint" "Package_DIP:DIP-14_W7.62mm"
 			(at 175.26 133.35 0)
 			(hide yes)
@@
 			)
 		)
-		(property "Footprint" ""
+		(property "Footprint" "LED_THT:LED_D5.0mm"
 			(at 203.2 113.03 0)
 			(hide yes)
@@
 			)
 		)
-		(property "Footprint" "Package_DIP:DIP-8_W7.62mm"
+		(property "Footprint" "Resistor_THT:R_Axial_DIN0204_L3.6mm_D1.6mm_P5.08mm_Horizontal"
 			(at 199.136 54.864 90)
 			(hide yes)
@@
 			)
 		)
-		(property "Footprint" "Package_SO:SOIC-8_3.9x4.9mm_P1.27mm"
+		(property "Footprint" "Capacitor_THT:C_Disc_D5.0mm_W2.5mm_P2.50mm"
 			(at 62.23 26.9748 0)
 			(hide yes)
@@
 			)
 		)
-		(property "Footprint" ""
+		(property "Footprint" "LED_THT:LED_D5.0mm"
 			(at 185.42 62.23 0)
 			(hide yes)
@@
 			)
 		)
-		(property "Footprint" ""
+		(property "Footprint" "LED_THT:LED_D5.0mm"
 			(at 154.94 147.32 0)
 			(hide yes)
@@
 			)
 		)
-		(property "Footprint" ""
+		(property "Footprint" "Resistor_THT:R_Axial_DIN0204_L3.6mm_D1.6mm_P5.08mm_Horizontal"
 			(at 81.534 22.606 90)
 			(hide yes)
@@
 			)
 		)
-		(property "Footprint" "Package_TO_SOT_SMD:SOT-363_SC-70-6"
+		(property "Footprint" "Package_DIP:DIP-16_W7.62mm"
 			(at 129.54 71.12 0)
 			(hide yes)
@@
 			)
 		)
-		(property "Footprint" "Package_SO:SSOP-24_5.3x8.2mm_P0.65mm"
+		(property "Footprint" "Package_DIP:DIP-14_W7.62mm"
 			(at 175.26 86.36 0)
 			(hide yes)
@@
 			)
 		)
-		(property "Footprint" ""
+		(property "Footprint" "Resistor_THT:R_Axial_DIN0204_L3.6mm_D1.6mm_P5.08mm_Horizontal"
 			(at 74.676 25.146 90)
 			(hide yes)
@@
 			)
 		)
-		(property "Footprint" ""
+		(property "Footprint" "LED_THT:LED_D5.0mm"
 			(at 198.12 62.23 0)
 			(hide yes)
@@
 			)
 		)
-		(property "Footprint" "Package_SO:SSOP-24_5.3x8.2mm_P0.65mm"
+		(property "Footprint" "Package_DIP:DIP-14_W7.62mm"
 			(at 175.26 101.6 0)
 			(hide yes)

Commit message: start PCB
Parts:
- BT1: footprint Battery:BatteryHolder_Keystone_1060_1x2032 -> Battery:BatteryHolder_Keystone_103_1x20mm
- renumbered D7 to D2, D2 to D4, D4 to D5, D5 to D7, R7 to R1, R3 to R10, R9 to R2, R6 to R3, R10 to R5, R8 to R6, R5 to R7, R1 to R8, R2 to R9
Changed lines of the file:
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@@
 		(dnp no)
 		(fields_autoplaced yes)
-		(property "Reference" "R7"
+		(property "Reference" "R1"
 			(at 205.74 104.1399 0)
 			(show_name no)
@@
 			(project "Dice"
 				(path "/468d8eab-55b6-4b88-919a-a10fe942a8e1"
-					(reference "R7")
+					(reference "R1")
 					(unit 1)
 				)
@@
 			)
 		)
-		(property "Footprint" "Battery:BatteryHolder_Keystone_1060_1x2032"
+		(property "Footprint" "Battery:BatteryHolder_Keystone_103_1x20mm"
 			(at 19.05 23.876 90)
 			(hide yes)
@@
 		(dnp no)
 		(fields_autoplaced yes)
-		(property "Reference" "R3"
+		(property "Reference" "R10"
 			(at 144.78 38.0999 0)
 			(show_name no)
@@
 			(project "Dice"
 				(path "/468d8eab-55b6-4b88-919a-a10fe942a8e1"
-					(reference "R3")
+					(reference "R10")
 					(unit 1)
 				)
@@
 		(dnp no)
 		(fields_autoplaced yes)
-		(property "Reference" "R9"
+		(property "Reference" "R2"
 			(at 189.23 135.8899 0)
 			(show_name no)
@@
 			(project "Dice"
 				(path "/468d8eab-55b6-4b88-919a-a10fe942a8e1"
-					(reference "R9")
+					(reference "R2")
 					(unit 1)
 				)
@@
 		(in_pos_files yes)
 		(dnp no)
-		(property "Reference" "R6"
+		(property "Reference" "R3"
 			(at 147.32 138.4299 0)
 			(show_name no)
@@
 			(project "Dice"
 				(path "/468d8eab-55b6-4b88-919a-a10fe942a8e1"
-					(reference "R6")
+					(reference "R3")
 					(unit 1)
 				)
@@
 		(in_pos_files yes)
 		(dnp no)
-		(property "Reference" "R8"
+		(property "Reference" "R6"
 			(at 157.48 138.4299 0)
 			(show_name no)
@@
 			(project "Dice"
 				(path "/468d8eab-55b6-4b88-919a-a10fe942a8e1"
-					(reference "R8")
+					(reference "R6")
 					(unit 1)
 				)
@@
 		(dnp no)
 		(fields_autoplaced yes)
-		(property "Reference" "D5"
+		(property "Reference" "D7"
 			(at 203.2 145.0974 90)
 			(show_name no)
@@
 			(project "Dice"
 				(path "/468d8eab-55b6-4b88-919a-a10fe942a8e1"
-					(reference "D5")
+					(reference "D7")
 					(unit 1)
 				)
@@
 		(dnp no)
 		(fields_autoplaced yes)
-		(property "Reference" "R5"
+		(property "Reference" "R7"
 			(at 201.93 135.8899 0)
 			(show_name no)
@@
 			(project "Dice"
 				(path "/468d8eab-55b6-4b88-919a-a10fe942a8e1"
-					(reference "R5")
+					(reference "R7")
 					(unit 1)
 				)
@@
 		(dnp no)
 		(fields_autoplaced yes)
-		(property "Reference" "D7"
+		(property "Reference" "D2"
 			(at 190.5 145.0974 90)
 			(show_name no)
@@
 			(project "Dice"
 				(path "/468d8eab-55b6-4b88-919a-a10fe942a8e1"
-					(reference "D7")
+					(reference "D2")
 					(unit 1)
 				)
@@
 		(dnp no)
 		(fields_autoplaced yes)
-		(property "Reference" "R10"
+		(property "Reference" "R5"
 			(at 200.66 53.3399 0)
 			(show_name no)
@@
 			(project "Dice"
 				(path "/468d8eab-55b6-4b88-919a-a10fe942a8e1"
-					(reference "R10")
+					(reference "R5")
 					(unit 1)
 				)
@@
 		(dnp no)
 		(fields_autoplaced yes)
-		(property "Reference" "D2"
+		(property "Reference" "D4"
 			(at 189.23 62.5474 90)
 			(show_name no)
@@
 			(project "Dice"
 				(path "/468d8eab-55b6-4b88-919a-a10fe942a8e1"
-					(reference "D2")
+					(reference "D4")
 					(unit 1)
 				)
@@
 		(dnp no)
 		(fields_autoplaced yes)
-		(property "Reference" "R2"
+		(property "Reference" "R9"
 			(at 85.09 21.5899 0)
 			(show_name no)
@@
 			(project "Dice"
 				(path "/468d8eab-55b6-4b88-919a-a10fe942a8e1"
-					(reference "R2")
+					(reference "R9")
 					(unit 1)
 				)
@@
 		(dnp no)
 		(fields_autoplaced yes)
-		(property "Reference" "R1"
+		(property "Reference" "R8"
 			(at 74.93 17.78 90)
 			(show_name no)
@@
 			(project "Dice"
 				(path "/468d8eab-55b6-4b88-919a-a10fe942a8e1"
-					(reference "R1")
+					(reference "R8")
 					(unit 1)
 				)
@@
 		(dnp no)
 		(fields_autoplaced yes)
-		(property "Reference" "D4"
+		(property "Reference" "D5"
 			(at 201.93 62.5474 90)
 			(show_name no)
@@
 			(project "Dice"
 				(path "/468d8eab-55b6-4b88-919a-a10fe942a8e1"
-					(reference "D4")
+					(reference "D5")
 					(unit 1)
 				)

Commit message: Fix some detail on the schema
Connections:
- net at R3.1: now also R6.1, U2.1 (Q5), U3.13; no longer D3.2 (A)
- new net: D3.2 (A), R3.2
Other:
- moved on the sheet: R3
Changed lines of the file:
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@@
+	)
+	(junction
+		(at 144.78 135.89)
+		(diameter 0)
+		(color 0 0 0 0)
 	)
 	(junction
@@
 	)
 	(junction
-		(at 186.69 133.35)
+		(at 68.58 27.94)
 		(diameter 0)
 		(color 0 0 0 0)
 	)
 	(junction
-		(at 68.58 27.94)
+		(at 186.69 133.35)
 		(diameter 0)
 		(color 0 0 0 0)
@@
 	)
 	(junction
-		(at 144.78 135.89)
-		(diameter 0)
-		(color 0 0 0 0)
-	)
-	(junction
 		(at 154.94 135.89)
 		(diameter 0)
@@
 	(wire
 		(pts
+			(xy 186.69 133.35) (xy 199.39 133.35)
+		)
+		(stroke
+			(width 0)
+			(type default)
+		)
+	)
+	(wire
+		(pts
 			(xy 54.61 43.18) (xy 36.83 43.18)
 		)
@@
 	(wire
 		(pts
-			(xy 186.69 133.35) (xy 199.39 133.35)
-		)
-		(stroke
-			(width 0)
-			(type default)
-		)
-	)
-	(wire
-		(pts
 			(xy 127 86.36) (xy 101.6 86.36)
 		)
@@
 	(wire
 		(pts
+			(xy 144.78 135.89) (xy 154.94 135.89)
+		)
+		(stroke
+			(width 0)
+			(type default)
+		)
+	)
+	(wire
+		(pts
 			(xy 162.56 43.18) (xy 162.56 83.82)
 		)
@@
 		(pts
 			(xy 73.66 54.61) (xy 73.66 53.34)
-		)
-		(stroke
-			(width 0)
-			(type default)
-		)
-	)
-	(wire
-		(pts
-			(xy 144.78 135.89) (xy 154.94 135.89)
 		)
 		(stroke
@@
 	(symbol
 		(lib_id "Device:R_US")
-		(at 144.78 139.7 180)
+		(at 144.78 139.7 0)
 		(unit 1)
 		(body_style 1)
@@
 		(dnp no)
 		(property "Reference" "R3"
-			(at 147.32 138.4299 0)
+			(at 142.24 140.9701 0)
 			(show_name no)
 			(do_not_autoplace no)
@@
 		)
 		(property "Value" "1k"
-			(at 147.32 140.9699 0)
+			(at 142.24 138.4301 0)
 			(show_name no)
 			(do_not_autoplace no)
@@
 		)
 		(property "Footprint" "Resistor_THT:R_Axial_DIN0204_L3.6mm_D1.6mm_P5.08mm_Horizontal"
-			(at 143.764 139.446 90)
-			(hide yes)
-			(show_name no)
+			(at 145.796 139.954 90)
+			(hide yes)
+			(show_name no)

Commit message: Creation of the PCB
Connections:
- net at C1.2, U1.2 (TRIG), U1.6 (THRES): now also R8.1; no longer R8.2
- net at R9.1, U1.7 (DISCH): now also R8.2; no longer R8.1
Other:
- moved on the sheet: R8
Changed lines of the file:
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@@
 	(symbol
 		(lib_id "Device:R_US")
-		(at 74.93 24.13 270)
+		(at 74.93 24.13 90)
 		(unit 1)
 		(body_style 1)
@@
 		)
 		(property "Footprint" "Resistor_THT:R_Axial_DIN0204_L3.6mm_D1.6mm_P5.08mm_Horizontal"
-			(at 74.676 25.146 90)
+			(at 75.184 23.114 90)
 			(hide yes)
 			(show_name no)

Commit message: addaed a a footrpiont and symbol for the button
Parts:
- removed SW2: SW_DPST_x2, Button_Switch_THT:SW_DIP_SPSTx01_Slide_9.78x4.72mm_W7.62mm_P2.54mm, symbol Switch:SW_DPST_x2
- added S1: EVQ-P0E07K, footprints:EVQP0E07K, symbol symbols:EVQ-P0E07K
Connections:
- net +3V: now also S1.A1 (COM)
- net at BT1.1 (+): now also S1.B1 (NO)
Changed lines of the file:
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@@
 	(wire
 		(pts
+			(xy 19.05 20.32) (xy 30.48 20.32)
+		)
+		(stroke
+			(width 0)
+			(type default)
+		)
+	)
+	(wire
+		(pts
 			(xy 154.94 135.89) (xy 167.64 135.89)
 		)
@@
 	(wire
 		(pts
-			(xy 19.05 20.32) (xy 30.48 20.32)
-		)
-		(stroke
-			(width 0)
-			(type default)
-		)
-	)
-	(wire
-		(pts
 			(xy 182.88 123.19) (xy 167.64 123.19)
 		)
@@
 	)
 	(symbol
-		(lib_id "Switch:SW_DPST_x2")
-		(at 35.56 20.32 0)
-		(unit 1)
-		(body_style 1)
-		(exclude_from_sim no)
-		(in_bom yes)
-		(on_board yes)
-		(in_pos_files yes)
-		(dnp no)
-		(fields_autoplaced yes)
-		(property "Reference" "SW2"
-			(at 35.56 13.97 0)
-			(show_name no)
-			(do_not_autoplace no)
-			(effects
-				(font
-					(size 1.27 1.27)
-				)
-			)
-		)
-		(property "Value" "SW_DPST_x2"
-			(at 35.56 16.51 0)
-			(show_name no)
-			(do_not_autoplace no)
-			(effects
-				(font
-					(size 1.27 1.27)
-				)
-			)
-		)
-		(property "Footprint" "Button_Switch_THT:SW_DIP_SPSTx01_Slide_9.78x4.72mm_W7.62mm_P2.54mm"
-			(at 35.56 20.32 0)
-			(hide yes)
-			(show_name no)
-			(do_not_autoplace no)
-			(effects
-				(font
-					(size 1.27 1.27)
-				)
-			)
-		)
-		(property "Datasheet" ""
-			(at 35.56 20.32 0)
-			(hide yes)
-			(show_name no)
-			(do_not_autoplace no)
-			(effects
-				(font
-					(size 1.27 1.27)
-				)
-			)
-		)
-		(property "Description" "Single Pole Single Throw (SPST) switch, separate symbol"
-			(at 35.56 20.32 0)
-			(hide yes)
-			(show_name no)
-			(do_not_autoplace no)
-			(effects
-				(font
-					(size 1.27 1.27)
-				)
-			)
-		)
-		(pin "1"
-		)
-		(pin "3"
-		)
-		(pin "2"
-		)
-		(pin "4"
-		)
-		(instances
-			(project "Dice"
-				(path "/468d8eab-55b6-4b88-919a-a10fe942a8e1"
-					(reference "SW2")
-					(unit 1)
-				)
-			)
-		)
-	)
-	(symbol
 		(lib_id "power:GND")
 		(at 139.7 58.42 180)
@@
 	)
 	(symbol
+		(lib_id "symbols:EVQ-P0E07K")
+		(at 30.48 17.78 0)
+		(unit 1)
+		(body_style 1)
+		(exclude_from_sim no)
+		(in_bom yes)
+		(on_board yes)
+		(in_pos_files yes)
+		(dnp no)
+		(property "Reference" "S1"
+			(at 48.768 18.288 0)
+			(show_name no)
+			(do_not_autoplace no)
+			(effects
+				(font
+					(size 1.27 1.27)
+				)
+				(justify left)
+			)
+		)
+		(property "Value" "EVQ-P0E07K"
+			(at 35.814 24.13 0)
+			(show_name no)
+			(do_not_autoplace no)
+			(effects
+				(font
+					(size 1.27 1.27)
+				)
+				(justify left)
+			)
+		)
+		(property "Footprint" "footprints:EVQP0E07K"
+			(at 49.53 112.7 0)
+			(hide yes)
+			(show_name no)
+			(do_not_autoplace no)
+			(effects
+				(font
+					(size 1.27 1.27)
+				)
+				(justify left top)
+			)
+		)
+		(property "Datasheet" "https://4donline.ihs.com/images/VipMasterIC/IC/PANA/PANAS38644/PANAS38644-1.pdf?hkey=52A5661711E402568146F3353EA87419"
+			(at 49.53 212.7 0)
+			(hide yes)
+			(show_name no)
+			(do_not_autoplace no)
+			(effects
+				(font
+					(size 1.27 1.27)
+				)
+				(justify left top)
+			)
+		)
+		(property "Description" "Black Tactile Switch, Single Pole Single Throw (SPST) 50 mA @ 30 V dc 7.45mm"
+			(at 30.48 17.78 0)
+			(hide yes)
+			(show_name no)
+			(do_not_autoplace no)
+			(effects
+				(font
+					(size 1.27 1.27)
+				)
+			)
+		)
+		(property "Height" "7.45"
+			(at 49.53 412.7 0)
+			(hide yes)
+			(show_name no)
+			(do_not_autoplace no)
+			(effects
+				(font
+					(size 1.27 1.27)
+				)
+				(justify left top)
+			)
+		)
+		(property "Mouser Part Number" "667-EVQ-P0E07K"
+			(at 49.53 512.7 0)
+			(hide yes)
+			(show_name no)
+			(do_not_autoplace no)
+			(effects
+				(font
+					(size 1.27 1.27)
+				)
+				(justify left top)
+			)
+		)
+		(property "Mouser Price/Stock" "https://www.mouser.co.uk/ProductDetail/Panasonic/EVQ-P0E07K?qs=EER3j8OP4JjRBsW%252BCEIoOg%3D%3D"
+			(at 49.53 612.7 0)
+			(hide yes)
+			(show_name no)
+			(do_not_autoplace no)
+			(effects
+				(font
+					(size 1.27 1.27)
+				)
+				(justify left top)
+			)
+		)
+		(property "Manufacturer_Name" "Panasonic"
+			(at 49.53 712.7 0)
+			(hide yes)
+			(show_name no)
+			(do_not_autoplace no)
+			(effects
+				(font
+					(size 1.27 1.27)
+				)
+				(justify left top)
+			)
+		)
+		(property "Manufacturer_Part_Number" "EVQ-P0E07K"
+			(at 49.53 812.7 0)
+			(hide yes)
+			(show_name no)
+			(do_not_autoplace no)
+			(effects
+				(font
+					(size 1.27 1.27)
+				)
+				(justify left top)
+			)
+		)
+		(pin "B1"
+		)
+		(pin "A1"
+		)
+		(instances
+			(project "Dice"
+				(path "/468d8eab-55b6-4b88-919a-a10fe942a8e1"
+					(reference "S1")
+					(unit 1)
+				)
+			)
+		)
+	)
+	(symbol
 		(lib_id "power:GND")
 		(at 185.42 66.04 0)
@@
 	(symbol
 		(lib_id "power:+5V")
-		(at 40.64 20.32 270)
+		(at 30.48 17.78 90)
 		(unit 1)
 		(body_style 1)
@@
 		(fields_autoplaced yes)
 		(property "Reference" "#PWR021"
-			(at 36.83 20.32 0)
+			(at 34.29 17.78 0)
 			(hide yes)
 			(show_name no)
@@
 		)
 		(property "Value" "+3V"
-			(at 44.45 20.3199 90)
+			(at 29.21 15.24 90)
 			(show_name no)
 			(do_not_autoplace no)
@@
 					(size 1.27 1.27)
 				)
-				(justify left)
 			)
 		)
 		(property "Footprint" ""
-			(at 40.64 20.32 0)
+			(at 30.48 17.78 0)
 			(hide yes)
 			(show_name no)
@@
 		)
 		(property "Datasheet" ""
-			(at 40.64 20.32 0)
+			(at 30.48 17.78 0)
 			(hide yes)
 			(show_name no)
@@
 		)
 		(property "Description" "Power symbol creates a global label with name \"+5V\""
-			(at 40.64 20.32 0)
+			(at 30.48 17.78 0)
 			(hide yes)
 			(show_name no)
