File: Dice.kicad_sch (KiCad schematic)
At the start: 27 parts, among them Q1 NPN, SW1 SW_Push, U1 LM555xM, U2 4017, U3 74LS32

Commit message: Added a secutiry diodo
Parts:
- added D8: D, Diode_THT:D_DO-41_SOD81_P10.16mm_Horizontal, symbol Device:D
Connections:
- net at BT1.1 (+): now also D8.2 (A); no longer S1.B1 (NO)
- new net: D8.1 (K), S1.B1 (NO)
Other:
- moved on the sheet: S1
Changed lines of the file:
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@@
 	(wire
 		(pts
-			(xy 19.05 20.32) (xy 30.48 20.32)
-		)
-		(stroke
-			(width 0)
-			(type default)
-		)
-	)
-	(wire
-		(pts
 			(xy 154.94 135.89) (xy 167.64 135.89)
 		)
@@
 	(wire
 		(pts
+			(xy 31.75 20.32) (xy 36.83 20.32)
+		)
+		(stroke
+			(width 0)
+			(type default)
+		)
+	)
+	(wire
+		(pts
 			(xy 54.61 27.94) (xy 54.61 43.18)
 		)
@@
 	(wire
 		(pts
+			(xy 19.05 20.32) (xy 24.13 20.32)
+		)
+		(stroke
+			(width 0)
+			(type default)
+		)
+	)
+	(wire
+		(pts
 			(xy 68.58 27.94) (xy 68.58 33.02)
 		)
@@
 	(symbol
 		(lib_id "symbols:EVQ-P0E07K")
-		(at 30.48 17.78 0)
+		(at 36.83 17.78 0)
 		(unit 1)
 		(body_style 1)
@@
 		(dnp no)
 		(property "Reference" "S1"
-			(at 48.768 18.288 0)
+			(at 55.118 18.288 0)
 			(show_name no)
 			(do_not_autoplace no)
@@
 		)
 		(property "Value" "EVQ-P0E07K"
-			(at 35.814 24.13 0)
+			(at 42.164 24.13 0)
 			(show_name no)
 			(do_not_autoplace no)
@@
 		)
 		(property "Footprint" "footprints:EVQP0E07K"
-			(at 49.53 112.7 0)
+			(at 55.88 112.7 0)
 			(hide yes)
 			(show_name no)
@@
 		)
 		(property "Datasheet" "https://4donline.ihs.com/images/VipMasterIC/IC/PANA/PANAS38644/PANAS38644-1.pdf?hkey=52A5661711E402568146F3353EA87419"
-			(at 49.53 212.7 0)
+			(at 55.88 212.7 0)
 			(hide yes)
 			(show_name no)
@@
 		)
 		(property "Description" "Black Tactile Switch, Single Pole Single Throw (SPST) 50 mA @ 30 V dc 7.45mm"
-			(at 30.48 17.78 0)
+			(at 36.83 17.78 0)
 			(hide yes)
 			(show_name no)
@@
 		)
 		(property "Height" "7.45"
-			(at 49.53 412.7 0)
+			(at 55.88 412.7 0)
 			(hide yes)
 			(show_name no)
@@
 		)
 		(property "Mouser Part Number" "667-EVQ-P0E07K"
-			(at 49.53 512.7 0)
+			(at 55.88 512.7 0)
 			(hide yes)
 			(show_name no)
@@
 		)
 		(property "Mouser Price/Stock" "https://www.mouser.co.uk/ProductDetail/Panasonic/EVQ-P0E07K?qs=EER3j8OP4JjRBsW%252BCEIoOg%3D%3D"
-			(at 49.53 612.7 0)
+			(at 55.88 612.7 0)
 			(hide yes)
 			(show_name no)
@@
 		)
 		(property "Manufacturer_Name" "Panasonic"
-			(at 49.53 712.7 0)
+			(at 55.88 712.7 0)
 			(hide yes)
 			(show_name no)
@@
 		)
 		(property "Manufacturer_Part_Number" "EVQ-P0E07K"
-			(at 49.53 812.7 0)
+			(at 55.88 812.7 0)
 			(hide yes)
 			(show_name no)
@@
 	(symbol
 		(lib_id "power:+5V")
-		(at 30.48 17.78 90)
+		(at 36.83 17.78 90)
 		(unit 1)
 		(body_style 1)
@@
 		(fields_autoplaced yes)
 		(property "Reference" "#PWR021"
-			(at 34.29 17.78 0)
+			(at 40.64 17.78 0)
 			(hide yes)
 			(show_name no)
@@
 		)
 		(property "Value" "+3V"
-			(at 29.21 15.24 90)
+			(at 35.56 15.24 90)
 			(show_name no)
 			(do_not_autoplace no)
@@
 		)
 		(property "Footprint" ""
-			(at 30.48 17.78 0)
+			(at 36.83 17.78 0)
 			(hide yes)
 			(show_name no)
@@
 		)
 		(property "Datasheet" ""
-			(at 30.48 17.78 0)
+			(at 36.83 17.78 0)
 			(hide yes)
 			(show_name no)
@@
 		)
 		(property "Description" "Power symbol creates a global label with name \"+5V\""
-			(at 30.48 17.78 0)
+			(at 36.83 17.78 0)
 			(hide yes)
 			(show_name no)
@@
 					(unit 1)
 				)
+			)
+		)
+	)
+	(symbol
+		(lib_id "Device:D")
+		(at 27.94 20.32 180)
+		(unit 1)
+		(body_style 1)
+		(exclude_from_sim no)
+		(in_bom yes)
+		(on_board yes)
+		(in_pos_files yes)
+		(dnp no)
+		(fields_autoplaced yes)
+		(property "Reference" "D8"
+			(at 27.94 13.97 0)
+			(show_name no)
+			(do_not_autoplace no)
+			(effects
+				(font
+					(size 1.27 1.27)
+				)
+			)
+		)
+		(property "Value" "D"
+			(at 27.94 16.51 0)
+			(show_name no)
+			(do_not_autoplace no)
+			(effects
+				(font
+					(size 1.27 1.27)
+				)
+			)
+		)
+		(property "Footprint" "Diode_THT:D_DO-41_SOD81_P10.16mm_Horizontal"
+			(at 27.94 20.32 0)
+			(hide yes)
+			(show_name no)
+			(do_not_autoplace no)
+			(effects
+				(font
+					(size 1.27 1.27)
+				)
+			)
+		)
+		(property "Datasheet" ""
+			(at 27.94 20.32 0)
+			(hide yes)
+			(show_name no)
+			(do_not_autoplace no)
+			(effects
+				(font
+					(size 1.27 1.27)
+				)
+			)
+		)
+		(property "Description" "Diode"
+			(at 27.94 20.32 0)
+			(hide yes)
+			(show_name no)
+			(do_not_autoplace no)
+			(effects
+				(font
+					(size 1.27 1.27)
+				)
+			)
+		)
+		(property "Sim.Device" "D"
+			(at 27.94 20.32 0)
+			(hide yes)
+			(show_name no)
+			(do_not_autoplace no)
+			(effects
+				(font
+					(size 1.27 1.27)
+				)
+			)
+		)
+		(property "Sim.Pins" "1=K 2=A"
+			(at 27.94 20.32 0)
+			(hide yes)
+			(show_name no)
+			(do_not_autoplace no)
+			(effects
+				(font
+					(size 1.27 1.27)
+				)
+			)
+		)
+		(pin "2"
+		)
+		(pin "1"
+		)
+		(instances
+			(project "Dice"
+				(path "/468d8eab-55b6-4b88-919a-a10fe942a8e1"
+					(reference "D8")
+					(unit 1)
+				)
