File: Dice.kicad_pcb (KiCad board)
At the start: 2 copper layers, 81.6 x 48.2 mm, 27 parts, among them Q1 NPN, SW1 SW_Push, SW2 SW_DPST_x2, U1 LM555xM, U2 4017, U3 74LS32

Commit message: Creation of the PCB
Parts:
- moved R10 50.8 mm to (86.0, 74.2), turned to 90 degrees
- moved Q1 39.2 mm to (123.9, 69.5), turned to 180 degrees
- moved U2 38.6 mm to (91.0, 76.1), turned to 90 degrees
- moved R1 34.5 mm to (123.5, 93.8), turned to 0 degrees
- moved R12 30.9 mm to (127.1, 69.2), turned to 0 degrees
- moved R7 30.0 mm to (123.7, 97.9), turned to 0 degrees
- moved R6 26.5 mm to (102.5, 89.0), turned to 0 degrees
- moved R3 17.6 mm to (102.5, 84.6), turned to 0 degrees
- moved R11 17.4 mm to (113.1, 69.2), turned to 0 degrees
- moved R5 14.4 mm to (127.6, 75.3)
- moved R4 14.4 mm to (124.0, 75.3)
- moved R2 12.7 mm to (102.4, 80.5), turned to 0 degrees
- moved U3 12.3 mm to (118.5, 102.8), turned to -90 degrees
- moved R8 4.74 mm to (86.0, 91.4), turned to 90 degrees
- moved D7 2.98 mm to (135.5, 95.1), turned to 180 degrees
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Connections:
- R3 pad 1: Net-(D3-A) -> Net-(U2-Q5)
- R3 pad 2: Net-(U2-Q5) -> Net-(D3-A)
- R8 pad 1: Net-(U1-DISCH) -> Net-(U1-THRES)
- R8 pad 2: Net-(U1-THRES) -> Net-(U1-DISCH)
Routing:
- net +3V: track 0.00 -> 158.1 mm, vias 0 -> 1
- net Net-(U2-Q0): track 0.00 -> 55.7 mm
- net Net-(R2-Pad1): track 0.00 -> 55.3 mm, vias 0 -> 1
- net Net-(U2-Q5): track 0.00 -> 54.8 mm, vias 0 -> 1
- net Net-(U2-Q2): track 0.00 -> 45.7 mm, vias 0 -> 1
- net Net-(U2-Q4): track 0.00 -> 44.6 mm
- net Net-(U2-Q3): track 0.00 -> 35.0 mm
- net Net-(U1-OUT): track 0.00 -> 27.7 mm
- net Net-(U1-THRES): track 0.00 -> 26.7 mm
- net Net-(U1-GND): track 0.00 -> 26.6 mm
- net Net-(D6-A): track 0.00 -> 26.6 mm
- net Net-(R1-Pad1): track 0.00 -> 22.3 mm
- net Net-(D4-A): track 0.00 -> 18.5 mm
- net Net-(U2-Q6): track 0.00 -> 15.1 mm
- net Net-(Q1-C): track 0.00 -> 12.9 mm
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
Commit message: Commit before braking changes
Other:
- board text added: "First Project"
Changed lines of the file:
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@@
 			(at 3.81 3.42 0)
 			(layer "F.Fab")
+			(hide yes)
 			(effects
 				(font
@@
 			(at 1.27 -3.56 0)
 			(layer "F.SilkS")
-			(hide yes)
 			(effects
 				(font
@@
 			(at 1.27 2.79 0)
 			(layer "F.Fab")
+			(hide yes)
 			(effects
 				(font
@@
 		)
 	)
+	(gr_poly
+		(pts
+			(xy 149.56 105.27) (xy 150.089167 109.900207) (xy 148.501667 107.915833) (xy 146.914167 109.900207)
+			(xy 147.443334 105.27) (xy 143.871459 101.962708) (xy 148.104792 103.682499) (xy 148.501667 102.624166)
+			(xy 148.898542 103.682499) (xy 153.131875 101.962708)
+		)
+		(stroke
+			(width 0.132291)
+			(type solid)
+		)
+		(fill yes)
+		(layer "F.SilkS")
+	)
 	(gr_rect
 		(start 81.75 65.5)
@@
 		(layer "Edge.Cuts")
 	)
+	(gr_text "First Project"
+		(at 141.47 99.88 0)
+		(layer "F.SilkS")
+		(effects
+			(font
+				(size 1.5 1.5)
+				(thickness 0.3)
+				(bold yes)
+			)
+			(justify left bottom)
+		)
+	)
 	(segment

Commit message: addaed a a footrpiont and symbol for the button
Parts:
- removed SW2: SW_DPST_x2, Button_Switch_THT:SW_DIP_SPSTx01_Slide_9.78x4.72mm_W7.62mm_P2.54mm
- added S1: EVQ-P0E07K, footprints:EVQP0E07K, F.Cu at (137.1, 70.2)
Routing:
- net Net-(BT1-+): track 6.98 -> 10.2 mm
- net +3V: track 158.1 -> 155.9 mm

Commit message: Added a secutiry diodo
Parts:
- added D8: D, Diode_THT:D_DO-41_SOD81_P10.16mm_Horizontal, F.Cu at (160.4, 107.3)
Connections:
- S1 pad B1: Net-(BT1-+) -> Net-(D8-K)
Routing:
- net Net-(D8-K): track 0.00 -> 44.7 mm
- net Net-(BT1-+): track 10.2 -> 33.3 mm

Commit message: Change the switch to turn on off
Parts:
- removed S1: EVQ-P0E07K, footprints:EVQP0E07K
- added SW2: SW_DPST_x2, Button_Switch_THT:SW_Slide-03_Wuerth-WS-SLTV_10x2.5x6.4_P2.54mm, F.Cu at (139.6, 70.2)
Routing:
- net Net-(D8-K): track 44.7 -> 45.8 mm
